File: hardware/keylink_revB/keylink_revB.kicad_pcb (KiCad board)
At the start: 2 copper layers, 23 x 40.5 mm, 7 parts, among them J1 Conn_01x02_Socket, J2 AudioJack3, SW1 SW_SPST, U1 XIAO ESP32C3

Commit message: Finalized revB.1 pcb
Parts:
- moved R2 17.6 mm to (96.1, 27.0)
- moved R1 17.1 mm to (96.1, 23.8)
- moved J1 11.6 mm to (96.8, 39.2), turned to 90 degrees
- moved C1 7.95 mm to (94.2, 32.8)
- moved J2 1.50 mm to (103.5, 26.0)
Connections:
- J2 pad R: Net-(U1-D1) -> Net-(U1-D6)
- J2 pad T: Net-(U1-D0) -> Net-(U1-D5)
- R1 pad 1: Net-(U1-D0) -> Net-(U1-D5)
- R2 pad 1: Net-(U1-D1) -> Net-(U1-D6)
- U1 pad 1: Net-(U1-D0) -> unconnected-(U1-D0-Pad1)
- U1 pad 2: Net-(U1-D1) -> unconnected-(U1-D1-Pad2)
- U1 pad 6: unconnected-(U1-D5-Pad6) -> Net-(U1-D5)
- U1 pad 7: unconnected-(U1-D6-Pad7) -> Net-(U1-D6)
Routing:
- net Net-(U1-D6): track 0.00 -> 57.3 mm
- net Net-(U1-VCC_3V3): track 0.00 -> 41.6 mm, vias 0 -> 1
- net Net-(U1-D5): track 0.00 -> 41.6 mm, vias 0 -> 1
- net Net-(J1-Pin_2): track 0.00 -> 24.6 mm, vias 0 -> 1
- net Net-(SW1-B): track 0.00 -> 21.6 mm
- net /VBAT: track 0.00 -> 8.51 mm
- net GND: track 0.00 -> 2.48 mm, vias 0 -> 5
- net unconnected-(U1-D1-Pad2): track 0.00 -> 1.08 mm
- net unconnected-(U1-D0-Pad1): track 0.00 -> 1.08 mm
- added copper zone on B.Cu, net GND
Other:
- outline, holes or cut-outs redrawn
- board text added: "MorseForge KeyLink rev b.1"
