File: hardware/keylink_revB/keylink_revB.kicad_sch (KiCad schematic)
At the start: 7 parts, among them J1 Conn_01x02_Socket, J2 AudioJack3, SW1 SW_Wuerth_450301014042, U1 XIAO ESP32C3

Commit message: Adding the pull up resistor footprints
Parts:
- R1, R2: footprint (none) -> Resistor_THT:R_Axial_DIN0207_L6.3mm_D2.5mm_P7.62mm_Horizontal
Changed lines of the file:
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@@
 			)
 		)
-		(property "Footprint" ""
+		(property "Footprint" "Resistor_THT:R_Axial_DIN0207_L6.3mm_D2.5mm_P7.62mm_Horizontal"
 			(at 153.162 44.45 90)
 			(effects
@@
 			)
 		)
-		(property "Footprint" ""
+		(property "Footprint" "Resistor_THT:R_Axial_DIN0207_L6.3mm_D2.5mm_P7.62mm_Horizontal"
 			(at 160.782 44.45 90)
 			(effects

Commit message: pcb layout completed
Parts:
- removed SW1: SW_Wuerth_450301014042, Button_Switch_THT:SW_Slide-03_Wuerth-WS-SLTV_10x2.5x6.4_P2.54mm, symbol Switch:SW_Wuerth_450301014042
- added SW1: SW_SPST, Button_Switch_THT:SW_Slide_SPDT_Angled_CK_OS102011MA1Q, symbol Switch:SW_SPST
- J1: footprint Connector_JST:JST_PH_B2B-PH-K_1x02_P2.00mm_Vertical -> Connector_JST:JST_PH_S2B-PH-K_1x02_P2.00mm_Horizontal
- J2: footprint Connector_Audio:Jack_3.5mm_PJ320D_Horizontal -> Connector_Audio:Jack_3.5mm_CUI_SJ1-3523N_Horizontal
Connections:
- net GND: now also U1.13 (GND)
- net VBAT: now also J1.1 (Pin_1), SW1.1 (A)
- net at U1.B+ (Batt+): now also SW1.2 (B)
- no-connect marks 0 -> 10

Commit message: Finalized revB.1 pcb
Connections:
- net at J2.T, R1.1: now also U1.6 (D5); no longer U1.1 (D0)
- net at J2.R, R2.1: now also U1.7 (D6); no longer U1.2 (D1)
Changed lines of the file:
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@@
-	)
-	(no_connect
-		(at 111.76 72.39)
 	)
 	(no_connect
@@
 	)
 	(no_connect
+		(at 111.76 53.34)
+	)
+	(no_connect
 		(at 147.32 60.96)
 	)
@@
 	)
 	(no_connect
-		(at 111.76 68.58)
+		(at 111.76 49.53)
 	)
 	(no_connect
@@
 	(wire
 		(pts
-			(xy 107.95 53.34) (xy 107.95 30.48)
-		)
-		(stroke
-			(width 0)
-			(type default)
-		)
-	)
-	(wire
-		(pts
 			(xy 189.23 64.77) (xy 179.07 64.77)
 		)
@@
 	(wire
 		(pts
-			(xy 111.76 49.53) (xy 111.76 34.29)
-		)
-		(stroke
-			(width 0)
-			(type default)
-		)
-	)
-	(wire
-		(pts
 			(xy 63.5 52.07) (xy 34.29 52.07)
 		)
@@
 	(wire
 		(pts
+			(xy 106.68 30.48) (xy 162.56 30.48)
+		)
+		(stroke
+			(width 0)
+			(type default)
+		)
+	)
+	(wire
+		(pts
 			(xy 154.94 34.29) (xy 154.94 40.64)
 		)
@@
 	(wire
 		(pts
-			(xy 107.95 30.48) (xy 162.56 30.48)
-		)
-		(stroke
-			(width 0)
-			(type default)
-		)
-	)
-	(wire
-		(pts
 			(xy 157.48 48.26) (xy 162.56 48.26)
 		)
@@
 	(wire
 		(pts
+			(xy 106.68 30.48) (xy 106.68 72.39)
+		)
+		(stroke
+			(width 0)
+			(type default)
+		)
+	)
+	(wire
+		(pts
+			(xy 106.68 72.39) (xy 111.76 72.39)
+		)
+		(stroke
+			(width 0)
+			(type default)
+		)
+	)
+	(wire
+		(pts
 			(xy 60.96 63.5) (xy 60.96 90.17)
 		)
@@
 	(wire
 		(pts
-			(xy 111.76 34.29) (xy 154.94 34.29)
+			(xy 107.95 34.29) (xy 154.94 34.29)
+		)
+		(stroke
+			(width 0)
+			(type default)
+		)
+	)
+	(wire
+		(pts
+			(xy 107.95 68.58) (xy 111.76 68.58)
+		)
+		(stroke
+			(width 0)
+			(type default)
+		)
+	)
+	(wire
+		(pts
+			(xy 107.95 34.29) (xy 107.95 68.58)
 		)
 		(stroke
@@
 		)
 		(stroke
-			(width 0)
-			(type default)
-		)
-	)
-	(wire
-		(pts
-			(xy 111.76 53.34) (xy 107.95 53.34)
-		)
-		(stroke
